Commit message: 修改模型

File: src/leo_description/urdf/d435.urdf.xacro (robot description, xacro)
@@ -9,5 +9,5 @@
     <link name="${name}_link">
       <visual>
-        <origin xyz="0 0 0" rpy="0 0 -1.5708"/>
+        <origin xyz="0 0 0" rpy="-1.5708 0 -1.5708"/>
         <geometry>
           <mesh filename="package://leo_description/models/d435.dae" />

File: src/leo_description/urdf/macros.xacro (robot description, xacro)
@@ -2,5 +2,5 @@
 <robot xmlns:xacro="http://www.ros.org/wiki/xacro">
   <xacro:include filename="$(find leo_description)/urdf/d435.urdf.xacro" />
-  <xacro:include filename="$(find leo_description)/urdf/mycobot_280_pi.xacro" />
+  <xacro:include filename="$(find leo_description)/urdf/mycobot_280_pi_adaptive_gripper.xacro" />
   <xacro:macro name="leo"
                params="default_antenna:=true

Commit message: 修改模型，指定配色与惯性矩阵

File: src/leo_description/urdf/d435.urdf.xacro (robot description, xacro)
@@ -32,7 +32,9 @@
     <link name="${name}_depth_optical_frame"/>
     <gazebo reference="${name}_link">
+      <material>Gazebo/Grey</material>
       <sensor name="${name}_rgbd" type="rgbd_camera">
         <camera>
-          <horizontal_fov>1.5184</horizontal_fov> <image>
+          <horizontal_fov>1.5184</horizontal_fov>
+          <image>
             <width>640</width>
             <height>480</height>
@@ -41,5 +43,6 @@
           <clip>
             <near>0.1</near>
-            <far>10.0</far> </clip>
+            <far>10.0</far>
+          </clip>
           <noise>
             <type>gaussian</type>

File: src/leo_description/urdf/mycobot_280_pi_adaptive_gripper.xacro (robot description, xacro)
@@ -1,194 +1,173 @@
-<?xml version="1.0"?>
+<?xml version="1.1"?>
 <robot xmlns:xacro="http://www.ros.org/wiki/xacro">
   <xacro:macro name="mycobot_280" params="parent prefix *origin">
-    <!-- 将父 link 连接到机械臂基座 -->
-    <joint name="${prefix}g_base_joint" type="fixed">
+    <xacro:macro name="cylinder_inertial" params="mass radius length">
+      <inertial>
+        <mass value="${mass * 10}"/>
+        <inertia
+          ixx="${(mass * 10) * (3 * radius * radius + length * length) / 12}" ixy="0.0" ixz="0.0"
+          iyy="${(mass * 10) * (3 * radius * radius + length * length) / 12}" iyz="0.0"
+          izz="${(mass * 10) * radius * radius / 2}" />
+      </inertial>
+    </xacro:macro>
+    <joint name="${prefix}base_to_parent" type="fixed">
       <xacro:insert_block name="origin" />
       <parent link="${parent}"/>
       <child link="${prefix}g_base"/>
     </joint>
-    <!-- 基座 link -->
     <link name="${prefix}g_base">
       <visual>
-        <geometry>
-          <mesh filename="package://mycobot_description/urdf/mycobot_280_pi/G_base.dae"/>
-        </geometry>
+        <geometry><mesh filename="package://leo_description/models/mycobot_280_pi/G_base.dae"/></geometry>
         <origin xyz="0.0 0 -0.03" rpy="0 0 1.5708"/>
       </visual>
       <collision>
-        <geometry>
-          <mesh filename="package://mycobot_description/urdf/mycobot_280_pi/G_base.dae"/>
-        </geometry>
+        <geometry><mesh filename="package://leo_description/models/mycobot_280_pi/G_base.dae"/></geometry>
         <origin xyz="0.0 0 -0.03" rpy="0 0 1.5708"/>
       </collision>
-    </link>
-    <!-- joint1 -->
+      <xacro:cylinder_inertial mass="0.5" radius="0.04" length="0.05"/>
+    </link>
     <link name="${prefix}joint1">
       <visual>
-        <geometry>
-          <mesh filename="package://mycobot_description/urdf/mycobot_280_pi/g_base_simple.stl"/>
-        </geometry>
+        <geometry><mesh filename="package://leo_description/models/mycobot_280_pi/g_base_simple.stl"/></geometry>
         <origin xyz="0.0 0 0" rpy="0 0 0"/>
       </visual>
       <collision>
-        <geometry>
-          <mesh filename="package://mycobot_description/urdf/mycobot_280_pi/g_base_simple.stl"/>
-        </geometry>
+        <geometry><mesh filename="package://leo_description/models/mycobot_280_pi/g_base_simple.stl"/></geometry>
         <origin xyz="0.0 0 0" rpy="0 0 0"/>
       </collision>
-    </link>
-    <joint name="${prefix}g_base_to_joint1" type="fixed">
-      <axis xyz="0 0 0"/>
-      <limit effort="1000.0" lower="-3.14" upper="3.14159" velocity="0"/>
+      <xacro:cylinder_inertial mass="0.2" radius="0.03" length="0.06"/>
+    </link>
+    <joint name="${prefix}g_base_to_joint1" type="revolute">
+      <axis xyz="0 0 1"/>
+      <limit effort="1000.0" lower="-3.14" upper="3.14159" velocity="1.0"/>
       <parent link="${prefix}g_base"/>
       <child link="${prefix}joint1"/>
       <origin xyz="0 0 0" rpy="0 0 0"/>
-    </joint>
-    <!-- joint2 -->
+      <dynamics damping="50.0" friction="50.0"/>
+    </joint>
     <link name="${prefix}joint2">
       <visual>
-        <geometry>
-          <mesh filename="package://mycobot_description/urdf/mycobot_280_pi/joint2.dae"/>
-        </geometry>
+        <geometry><mesh filename="package://leo_description/models/mycobot_280_pi/joint2.dae"/></geometry>
         <origin xyz="0.0 0 -0.06096" rpy="0 0 -1.5708"/>
       </visual>
       <collision>
-        <geometry>
-          <mesh filename="package://mycobot_description/urdf/mycobot_280_pi/joint2.dae"/>
-        </geometry>
+        <geometry><mesh filename="package://leo_description/models/mycobot_280_pi/joint2.dae"/></geometry>
         <origin xyz="0.0 0 -0.06096" rpy="0 0 -1.5708"/>
       </collision>
+      <xacro:cylinder_inertial mass="0.15" radius="0.02" length="0.1"/>
     </link>
     <joint name="${prefix}joint2_to_joint1" type="revolute">
       <axis xyz="0 0 1"/>
-      <limit effort="1000.0" lower="-2.9321" upper="2.9321" velocity="0"/>
+      <limit effort="1000.0" lower="-2.9321" upper="2.9321" velocity="1.0"/>
+      <origin xyz="0 0 0.13956" rpy="0 0 0"/>
       <parent link="${prefix}joint1"/>
       <child link="${prefix}joint2"/>
-      <origin xyz="0 0 0.13956" rpy="0 0 0"/>
-    </joint>
-    <!-- joint3 -->
+      <dynamics damping="50.0" friction="50.0"/>
+    </joint>
     <link name="${prefix}joint3">
       <visual>
-        <geometry>
-          <mesh filename="package://mycobot_description/urdf/mycobot_280_pi/joint3.dae"/>
-        </geometry>
+        <geometry><mesh filename="package://leo_description/models/mycobot_280_pi/joint3.dae"/></geometry>
         <origin xyz="0.0 0 0.03256" rpy="0 -1.5708 0"/>
       </visual>
       <collision>
-        <geometry>
-          <mesh filename="package://mycobot_description/urdf/mycobot_280_pi/joint3.dae"/>
-        </geometry>
+        <geometry><mesh filename="package://leo_description/models/mycobot_280_pi/joint3.dae"/></geometry>
         <origin xyz="0.0 0 0.03256" rpy="0 -1.5708 0"/>
       </collision>
+      <xacro:cylinder_inertial mass="0.15" radius="0.02" length="0.1"/>
     </link>
     <joint name="${prefix}joint3_to_joint2" type="revolute">
       <axis xyz="0 0 1"/>
-      <limit effort="1000.0" lower="-2.4434" upper="2.4434" velocity="0"/>
+      <limit effort="1000.0" lower="-2.4434" upper="2.4434" velocity="1.0"/>
+      <origin xyz="0 0 -0.001" rpy="0 1.5708 -1.5708"/>
       <parent link="${prefix}joint2"/>
       <child link="${prefix}joint3"/>
-      <origin xyz="0 0 -0.001" rpy="0 1.5708 -1.5708"/>
-    </joint>
-    <!-- joint4 -->
+      <dynamics damping="50.0" friction="50.0"/>
+    </joint>
     <link name="${prefix}joint4">
       <visual>
-        <geometry>
-          <mesh filename="package://mycobot_description/urdf/mycobot_280_pi/joint4.dae"/>
-        </geometry>
+        <geometry><mesh filename="package://leo_description/models/mycobot_280_pi/joint4.dae"/></geometry>
         <origin xyz="0.0 0 0.03056" rpy="0 -1.5708 0"/>
       </visual>
       <collision>
-        <geometry>
-          <mesh filename="package://mycobot_description/urdf/mycobot_280_pi/joint4.dae"/>
-        </geometry>
+        <geometry><mesh filename="package://leo_description/models/mycobot_280_pi/joint4.dae"/></geometry>
         <origin xyz="0.0 0 0.03056" rpy="0 -1.5708 0"/>
       </collision>
+      <xacro:cylinder_inertial mass="0.1" radius="0.02" length="0.05"/>
     </link>
     <joint name="${prefix}joint4_to_joint3" type="revolute">
       <axis xyz="0 0 1"/>
-      <limit effort="1000.0" lower="-2.6179" upper="2.6179" velocity="0"/>
+      <limit effort="1000.0" lower="-2.6179" upper="2.6179" velocity="1.0"/>
       <parent link="${prefix}joint3"/>
       <child link="${prefix}joint4"/>
       <origin xyz="-0.1104 0 0" rpy="0 0 0"/>
-    </joint>
-    <!-- joint5 -->
+      <dynamics damping="50.0" friction="50.0"/>
+    </joint>
     <link name="${prefix}joint5">
       <visual>
-        <geometry>
-          <mesh filename="package://mycobot_description/urdf/mycobot_280_pi/J5_simple.stl"/>
-        </geometry>
+        <geometry><mesh filename="package://leo_description/models/mycobot_280_pi/J5_simple.stl"/></geometry>
         <origin xyz="-0.02 0.002 0" rpy="0 0 0"/>
       </visual>
       <collision>
-        <geometry>
-          <mesh filename="package://mycobot_description/urdf/mycobot_280_pi/J5_simple.stl"/>
-        </geometry>
+        <geometry><mesh filename="package://leo_description/models/mycobot_280_pi/J5_simple.stl"/></geometry>
         <origin xyz="-0.02 0.002 0" rpy="0 0 0"/>
       </collision>
+      <xacro:cylinder_inertial mass="0.1" radius="0.02" length="0.05"/>
     </link>
     <joint name="${prefix}joint5_to_joint4" type="revolute">
       <axis xyz="0 0 1"/>
-      <limit effort="1000.0" lower="-2.6179" upper="2.6179" velocity="0"/>
+      <limit effort="1000.0" lower="-2.6179" upper="2.6179" velocity="1.0"/>
       <parent link="${prefix}joint4"/>
       <child link="${prefix}joint5"/>
       <origin xyz="-0.096 0 0.06462" rpy="0 0 -1.5708"/>
-    </joint>
-    <!-- joint6 -->
+      <dynamics damping="50.0" friction="50.0"/>
+    </joint>
     <link name="${prefix}joint6">
       <visual>
-        <geometry>
-          <mesh filename="package://mycobot_description/urdf/mycobot_280_pi/joint6.dae"/>
-        </geometry>
+        <geometry><mesh filename="package://leo_description/models/mycobot_280_pi/joint6.dae"/></geometry>
         <origin xyz="0 0.00 -0.038" rpy="0 0 0"/>
       </visual>
       <collision>
-        <geometry>
-          <mesh filename="package://mycobot_description/urdf/mycobot_280_pi/joint6.dae"/>
-        </geometry>
+        <geometry><mesh filename="package://leo_description/models/mycobot_280_pi/joint6.dae"/></geometry>
         <origin xyz="0 0.00 -0.038" rpy="0 0 0"/>
       </collision>
+      <xacro:cylinder_inertial mass="0.1" radius="0.02" length="0.04"/>
     </link>
     <joint name="${prefix}joint6_to_joint5" type="revolute">
       <axis xyz="0 0 1"/>
-      <limit effort="1000.0" lower="-2.7052" upper="2.7925" velocity="0"/>
+      <limit effort="1000.0" lower="-2.7052" upper="2.7925" velocity="1.0"/>
       <parent link="${prefix}joint5"/>
       <child link="${prefix}joint6"/>
       <origin xyz="0 -0.07318 -0.001" rpy="1.5708 -1.5708 0"/>
-    </joint>
-    <!-- joint6 flange -->
+      <dynamics damping="50.0" friction="50.0"/>
+    </joint>
     <link name="${prefix}joint6_flange">
       <visual>
-        <geometry>
-          <mesh filename="package://mycobot_description/urdf/mycobot_280_pi/joint7.dae"/>
-        </geometry>
+        <geometry><mesh filename="package://leo_description/models/mycobot_280_pi/joint7.dae"/></geometry>
         <origin xyz="0.0 0 -0.012" rpy="0 0 0"/>
       </visual>
       <collision>
-        <geometry>
-          <mesh filename="package://mycobot_description/urdf/mycobot_280_pi/joint7.dae"/>
-        </geometry>
+        <geometry><mesh filename="package://leo_description/models/mycobot_280_pi/joint7.dae"/></geometry>
         <origin xyz="0.0 0 -0.012" rpy="0 0 0"/>
       </collision>
+      <xacro:cylinder_inertial mass="0.05" radius="0.015" length="0.01"/>
     </link>
     <joint name="${prefix}joint6output_to_joint6" type="revolute">
       <axis xyz="0 0 1"/>
-      <limit effort="1000.0" lower="-3.14159" upper="3.14159" velocity="0"/>
+      <limit effort="1000.0" lower="-3.14159" upper="3.14159" velocity="1.0"/>
       <parent link="${prefix}joint6"/>
       <child link="${prefix}joint6_flange"/>
       <origin xyz="0 0.0456 0" rpy="-1.5708 0 0"/>
-    </joint>
-    <!-- 夹爪部分 -->
+      <dynamics damping="50.0" friction="50.0"/>
+    </joint>
     <link name="${prefix}gripper_base">
       <visual>
-        <geometry>
-          <mesh filename="package://mycobot_description/urdf/adaptive_gripper/gripper_base.dae"/>
-        </geometry>
+        <geometry><mesh filename="package://leo_description/models/adaptive_gripper/gripper_base.dae"/></geometry>
         <origin xyz="0.0 0 -0.012" rpy="0 0 0"/>
       </visual>
       <collision>
-        <geometry>
-          <mesh filename="package://mycobot_description/urdf/adaptive_gripper/gripper_base.dae"/>
-        </geometry>
+        <geometry><mesh filename="package://leo_description/models/adaptive_gripper/gripper_base.dae"/></geometry>
         <origin xyz="0.0 0 -0.012" rpy="0 0 0"/>
       </collision>
+      <xacro:cylinder_inertial mass="0.08" radius="0.03" length="0.03"/>
     </link>
     <joint name="${prefix}joint6output_to_gripper_base" type="fixed">
@@ -199,134 +178,166 @@
     <link name="${prefix}gripper_left1">
       <visual>
-        <geometry>
-          <mesh filename="package://mycobot_description/urdf/adaptive_gripper/gripper_left1.dae"/>
-        </geometry>
+        <geometry><mesh filename="package://leo_description/models/adaptive_gripper/gripper_left1.dae"/></geometry>
         <origin xyz="0.039 -0.0133 -0.012" rpy="0 0 0"/>
       </visual>
       <collision>
-        <geometry>
-          <mesh filename="package://mycobot_description/urdf/adaptive_gripper/gripper_left1.dae"/>
-        </geometry>
+        <geometry><mesh filename="package://leo_description/models/adaptive_gripper/gripper_left1.dae"/></geometry>
         <origin xyz="0.039 -0.0133 -0.012" rpy="0 0 0"/>
       </collision>
+      <xacro:cylinder_inertial mass="0.02" radius="0.01" length="0.02"/>
     </link>
     <link name="${prefix}gripper_left2">
       <visual>
-        <geometry>
-          <mesh filename="package://mycobot_description/urdf/adaptive_gripper/gripper_left2.dae"/>
-        </geometry>
+        <geometry><mesh filename="package://leo_description/models/adaptive_gripper/gripper_left2.dae"/></geometry>
         <origin xyz="0.005 -0.0195 -0.012" rpy="0 0 0"/>
       </visual>
       <collision>
-        <geometry>
-          <mesh filename="package://mycobot_description/urdf/adaptive_gripper/gripper_left2.dae"/>
-        </geometry>
+        <geometry><mesh filename="package://leo_description/models/adaptive_gripper/gripper_left2.dae"/></geometry>
         <origin xyz="0.005 -0.0195 -0.012" rpy="0 0 0"/>
       </collision>
+      <xacro:cylinder_inertial mass="0.02" radius="0.01" length="0.02"/>
     </link>
     <link name="${prefix}gripper_left3">
       <visual>
-        <geometry>
-          <mesh filename="package://mycobot_description/urdf/adaptive_gripper/gripper_left3.dae"/>
-        </geometry>
+        <geometry><mesh filename="package://leo_description/models/adaptive_gripper/gripper_left3.dae"/></geometry>
         <origin xyz="0.012 0.0025 -0.012" rpy="0 0 0"/>
       </visual>
       <collision>
-        <geometry>
-          <mesh filename="package://mycobot_description/urdf/adaptive_gripper/gripper_left3.dae"/>
-        </geometry>
+        <geometry><mesh filename="package://leo_description/models/adaptive_gripper/gripper_left3.dae"/></geometry>
         <origin xyz="0.012 0.0025 -0.012" rpy="0 0 0"/>
       </collision>
+      <xacro:cylinder_inertial mass="0.02" radius="0.01" length="0.03"/>
     </link>
     <link name="${prefix}gripper_right1">
       <visual>
-        <geometry>
-          <mesh filename="package://mycobot_description/urdf/adaptive_gripper/gripper_right1.dae"/>
-        </geometry>
+        <geometry><mesh filename="package://leo_description/models/adaptive_gripper/gripper_right1.dae"/></geometry>
         <origin xyz="-0.039 -0.0133 -0.012" rpy="0 0 0"/>
       </visual>
       <collision>
-        <geometry>
-          <mesh filename="package://mycobot_description/urdf/adaptive_gripper/gripper_right1.dae"/>
-        </geometry>
+        <geometry><mesh filename="package://leo_description/models/adaptive_gripper/gripper_right1.dae"/></geometry>
         <origin xyz="-0.039 -0.0133 -0.012" rpy="0 0 0"/>
       </collision>
+      <xacro:cylinder_inertial mass="0.02" radius="0.01" length="0.02"/>
     </link>
     <link name="${prefix}gripper_right2">
       <visual>
-        <geometry>
-          <mesh filename="package://mycobot_description/urdf/adaptive_gripper/gripper_right2.dae"/>
-        </geometry>
+        <geometry><mesh filename="package://leo_description/models/adaptive_gripper/gripper_right2.dae"/></geometry>
         <origin xyz="-0.005 -0.0195 -0.012" rpy="0 0 0"/>
       </visual>
       <collision>
-        <geometry>
-          <mesh filename="package://mycobot_description/urdf/adaptive_gripper/gripper_right2.dae"/>
-        </geometry>
+        <geometry><mesh filename="package://leo_description/models/adaptive_gripper/gripper_right2.dae"/></geometry>
         <origin xyz="-0.005 -0.0195 -0.012" rpy="0 0 0"/>
       </collision>
+      <xacro:cylinder_inertial mass="0.02" radius="0.01" length="0.02"/>
     </link>
     <link name="${prefix}gripper_right3">
       <visual>
-        <geometry>
-          <mesh filename="package://mycobot_description/urdf/adaptive_gripper/gripper_right3.dae"/>
-        </geometry>
+        <geometry><mesh filename="package://leo_description/models/adaptive_gripper/gripper_right3.dae"/></geometry>
         <origin xyz="-0.012 0.0025 -0.012" rpy="0 0 0"/>
       </visual>
       <collision>
-        <geometry>
-          <mesh filename="package://mycobot_description/urdf/adaptive_gripper/gripper_right3.dae"/>
-        </geometry>
+        <geometry><mesh filename="package://leo_description/models/adaptive_gripper/gripper_right3.dae"/></geometry>
         <origin xyz="-0.012 0.0025 -0.012" rpy="0 0 0"/>
       </collision>
-    </link>
-    <!-- 夹爪关节及 mimic 关系 -->
+      <xacro:cylinder_inertial mass="0.02" radius="0.01" length="0.02"/>
+    </link>
     <joint name="${prefix}gripper_controller" type="revolute">
       <axis xyz="0 0 1"/>
-      <limit effort="1000.0" lower="-0.74" upper="0.15" velocity="0"/>
+      <limit effort="1000.0" lower="-0.74" upper="0.15" velocity="1.0"/>
       <parent link="${prefix}gripper_base"/>
       <child link="${prefix}gripper_left3"/>
       <origin xyz="-0.012 0.005 0" rpy="0 0 0"/>
+      <dynamics damping="50.0" friction="50.0"/>
     </joint>
     <joint name="${prefix}gripper_base_to_gripper_left2" type="revolute">
       <axis xyz="0 0 1"/>
-      <limit effort="1000.0" lower="-0.8" upper="0.5" velocity="0"/>
+      <limit effort="1000.0" lower="-0.8" upper="0.5" velocity="1.0"/>
       <parent link="${prefix}gripper_base"/>
       <child link="${prefix}gripper_left2"/>
       <origin xyz="-0.005 0.027 0" rpy="0 0 0"/>
       <mimic joint="${prefix}gripper_controller" multiplier="1.0" offset="0"/>
+      <dynamics damping="50.0" friction="50.0"/>
     </joint>
     <joint name="${prefix}gripper_left3_to_gripper_left1" type="revolute">
       <axis xyz="0 0 1"/>
-      <limit effort="1000.0" lower="-0.5" upper="0.5" velocity="0"/>
+      <limit effort="1000.0" lower="-0.5" upper="0.5" velocity="1.0"/>
       <parent link="${prefix}gripper_left3"/>
       <child link="${prefix}gripper_left1"/>
       <origin xyz="-0.027 0.016 0" rpy="0 0 0"/>
       <mimic joint="${prefix}gripper_controller" multiplier="-1.0" offset="0"/>
+      <dynamics damping="50.0" friction="50.0"/>
     </joint>
     <joint name="${prefix}gripper_base_to_gripper_right3" type="revolute">
       <axis xyz="0 0 1"/>
-      <limit effort="1000.0" lower="-0.15" upper="0.7" velocity="0"/>
+      <limit effort="1000.0" lower="-0.15" upper="0.7" velocity="1.0"/>
       <parent link="${prefix}gripper_base"/>
       <child link="${prefix}gripper_right3"/>
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
Commit message: 更新相机模型xacro描述

File: src/leo_description/urdf/d435.urdf.xacro (robot description, xacro)
@@ -11,5 +11,5 @@
         <origin xyz="0 0 0" rpy="-1.5708 0 -1.5708"/>
         <geometry>
-          <mesh filename="package://leo_description/models/d435.dae" />
+          <mesh filename="package://leo_description/models/d435.stl" />
         </geometry>
       </visual>
