Commit message: Update simulation configurations

File: src/leo_description/urdf/macros.xacro (robot description, xacro)
@@ -1,4 +1,6 @@
 <?xml version="1.0" encoding="utf-8"?>
 <robot xmlns:xacro="http://www.ros.org/wiki/xacro">
+  <xacro:include filename="$(find leo_description)/urdf/d435.urdf.xacro" />
+  <xacro:include filename="$(find leo_description)/urdf/mycobot_280_pi.xacro" />
   <xacro:macro name="leo"
                params="default_antenna:=true
@@ -280,4 +282,10 @@
       <origin xyz="0.02313 0.0 -0.138" rpy="0.0 0.0 3.14"/>
     </joint>
+    <xacro:sensor_d435 parent="${link_prefix}base_link" name="${link_prefix}d435">
+      <origin xyz="0.17375 0.0 0.09568" rpy="0 0.34906 0"/>
+    </xacro:sensor_d435>
+    <xacro:mycobot_280 parent="${link_prefix}base_link" prefix="arm_">
+      <origin xyz="0.0995 0.0 0.032" rpy="0 0 0"/>
+    </xacro:mycobot_280>
   </xacro:macro>
   <!-- LEO GAZEBO -->

Commit message: 解决坐标冲突，添加仿真机械臂代码，创建总启动文件，修改导航启动文件

File: src/leo_description/urdf/macros.xacro (robot description, xacro)
@@ -249,10 +249,10 @@
       </joint>
     </xacro:if>
-    <joint name="${joint_prefix}camera_joint" type="fixed">
+    <joint name="${joint_prefix}leo_camera_joint" type="fixed">
       <origin xyz="0.0971 0 -0.0427" rpy="0 0.2094 0"/>
       <parent link="${link_prefix}base_link"/>
       <child link="${link_prefix}camera_frame"/>
     </joint>
-    <joint name="${joint_prefix}camera_optical_joint" type="fixed">
+    <joint name="${joint_prefix}leo_camera_optical_joint" type="fixed">
       <origin xyz="0 0 0" rpy="-${pi/2} 0.0 -${pi/2}"/>
       <parent link="${link_prefix}camera_frame"/>
@@ -282,6 +282,6 @@
       <origin xyz="0.02313 0.0 -0.138" rpy="0.0 0.0 3.14"/>
     </joint>
-    <xacro:sensor_d435 parent="${link_prefix}base_link" name="${link_prefix}d435">
-      <origin xyz="0.17375 0.0 0.09568" rpy="0 0.34906 0"/>
+    <xacro:sensor_d435 parent="${link_prefix}base_link" name="camera">
+    <origin xyz="0.17375 0.0 0.09568" rpy="0 0.34906 0"/>
     </xacro:sensor_d435>
     <xacro:mycobot_280 parent="${link_prefix}base_link" prefix="arm_">

Commit message: 修复视觉，更换坐标系，调整视觉与接近节点，构建机械臂节点

File: src/leo_description/urdf/macros.xacro (robot description, xacro)
@@ -254,5 +254,5 @@
       <child link="${link_prefix}camera_frame"/>
     </joint>
-    <joint name="${joint_prefix}leo_camera_optical_joint" type="fixed">
+    <joint name="${joint_prefix}camera_optical_joint" type="fixed">
       <origin xyz="0 0 0" rpy="-${pi/2} 0.0 -${pi/2}"/>
       <parent link="${link_prefix}camera_frame"/>
@@ -282,6 +282,6 @@
       <origin xyz="0.02313 0.0 -0.138" rpy="0.0 0.0 3.14"/>
     </joint>
-    <xacro:sensor_d435 parent="${link_prefix}base_link" name="camera">
-    <origin xyz="0.17375 0.0 0.09568" rpy="0 0.34906 0"/>
+    <xacro:sensor_d435 parent="${link_prefix}base_link" name="${link_prefix}camera">
+      <origin xyz="0.17375 0.0 0.09568" rpy="0 0.34906 0"/>
     </xacro:sensor_d435>
     <xacro:mycobot_280 parent="${link_prefix}base_link" prefix="arm_">
@@ -446,39 +446,4 @@
         </surface>
       </collision>
-    </gazebo>
-    <!-- camera -->
-    <gazebo reference="${link_prefix}camera_frame">
-      <sensor name="camera" type="camera">
-          <camera name="leo_camera">
-              <horizontal_fov>1.9</horizontal_fov>
-              <image>
-                  <width>640</width>
-                  <height>480</height>
-                  <format>R8G8B8</format>
-              </image>
-              <clip>
-                  <near>0.05</near>
-                  <far>300</far>
-              </clip>
-              <noise>
-                <type>gaussian</type>
-                <mean>0.0</mean>
-                <stddev>0.007</stddev>
-              </noise>
-              <distortion>
-                <k1>-0.279817</k1>
-                <k2>0.060321</k2>
-                <k3>0.000487</k3>
-                <p1>0.000310</p1>
-                <p2>0.000000</p2>
-                <center>0.5 0.5</center>
-              </distortion>
-          </camera>
-          <always_on>1</always_on>
-          <update_rate>30</update_rate>
-          <visualize>true</visualize>
-          <topic>${link_prefix}camera/image_raw</topic>
-          <gz_frame_id>${link_prefix}camera_optical_frame</gz_frame_id>
-      </sensor>
     </gazebo>
     <!-- rocker differential -->
