Commit message: 添加手臂配置以及简单运动测试

File: src/leo_description/urdf/mycobot_280_pi_adaptive_gripper.xacro (robot description, xacro)
@@ -340,4 +340,49 @@
       <material>Gazebo/DarkGrey</material>
     </gazebo>
+    <ros2_control name="ArmControlSystem" type="system">
+      <hardware>
+        <plugin>gz_ros2_control/GazeboSimSystem</plugin>
+      </hardware>
+      <joint name="${prefix}g_base_to_joint1">
+        <command_interface name="position"/>
+        <state_interface name="position"/>
+        <state_interface name="velocity"/>
+      </joint>
+      <joint name="${prefix}joint2_to_joint1">
+        <command_interface name="position"/>
+        <state_interface name="position"/>
+        <state_interface name="velocity"/>
+      </joint>
+      <joint name="${prefix}joint3_to_joint2">
+        <command_interface name="position"/>
+        <state_interface name="position"/>
+        <state_interface name="velocity"/>
+      </joint>
+      <joint name="${prefix}joint4_to_joint3">
+        <command_interface name="position"/>
+        <state_interface name="position"/>
+        <state_interface name="velocity"/>
+      </joint>
+      <joint name="${prefix}joint5_to_joint4">
+        <command_interface name="position"/>
+        <state_interface name="position"/>
+        <state_interface name="velocity"/>
+      </joint>
+      <joint name="${prefix}joint6_to_joint5">
+        <command_interface name="position"/>
+        <state_interface name="position"/>
+        <state_interface name="velocity"/>
+      </joint>
+      <joint name="${prefix}joint6output_to_joint6">
+        <command_interface name="position"/>
+        <state_interface name="position"/>
+        <state_interface name="velocity"/>
+      </joint>
+    </ros2_control>
+    <gazebo>
+      <plugin filename="gz_ros2_control-system" name="gz_ros2_control::GazeboSimROS2ControlPlugin">
+        <parameters>$(find leo_description)/config/arm_controller.yaml</parameters>
+      </plugin>
+    </gazebo>
   </xacro:macro>
 </robot>

Commit message: 创建新世界模型，修改模型，修改机械臂控制配置

File: src/leo_description/urdf/mycobot_280_pi_adaptive_gripper.xacro (robot description, xacro)
@@ -38,5 +38,5 @@
       <xacro:cylinder_inertial mass="0.2" radius="0.03" length="0.06"/>
     </link>
-    <joint name="${prefix}g_base_to_joint1" type="revolute">
+    <joint name="${prefix}g_base_to_joint1" type="fixed">
       <axis xyz="0 0 1"/>
       <limit effort="1000.0" lower="-3.14" upper="3.14159" velocity="1.0"/>

Commit message: 编写机械臂控制节点

File: src/leo_description/urdf/mycobot_280_pi_adaptive_gripper.xacro (robot description, xacro)
@@ -344,9 +344,4 @@
         <plugin>gz_ros2_control/GazeboSimSystem</plugin>
       </hardware>
-      <joint name="${prefix}g_base_to_joint1">
-        <command_interface name="position"/>
-        <state_interface name="position"/>
-        <state_interface name="velocity"/>
-      </joint>
       <joint name="${prefix}joint2_to_joint1">
         <command_interface name="position"/>

Commit message: 更换模型，调整体积

File: src/leo_description/urdf/mycobot_280_pi_adaptive_gripper.xacro (robot description, xacro)
@@ -22,5 +22,5 @@
       </visual>
       <collision>
-        <geometry><mesh filename="package://leo_description/models/mycobot_280_pi/G_base.dae"/></geometry>
+        <geometry><mesh filename="package://leo_description/models/mycobot_280_pi/G_base.dae" scale="0.9 0.9 0.9"/></geometry>
         <origin xyz="0.0 0 -0.03" rpy="0 0 1.5708"/>
       </collision>
@@ -29,10 +29,10 @@
     <link name="${prefix}joint1">
       <visual>
-        <geometry><mesh filename="package://leo_description/models/mycobot_280_pi/g_base_simple.stl"/></geometry>
-        <origin xyz="0.0 0 0" rpy="0 0 0"/>
-      </visual>
-      <collision>
-        <geometry><mesh filename="package://leo_description/models/mycobot_280_pi/g_base_simple.stl"/></geometry>
-        <origin xyz="0.0 0 0" rpy="0 0 0"/>
+        <geometry><mesh filename="package://leo_description/models/mycobot_280_pi/joint1.dae"/></geometry>
+        <origin xyz="0.0 0 0" rpy="0 0 -1.5708"/>
+      </visual>
+      <collision>
+        <geometry><mesh filename="package://leo_description/models/mycobot_280_pi/joint1.dae" scale="0.9 0.9 0.9"/></geometry>
+        <origin xyz="0.0 0 0" rpy="0 0 -1.5708"/>
       </collision>
       <xacro:cylinder_inertial mass="0.2" radius="0.03" length="0.06"/>
@@ -52,5 +52,5 @@
       </visual>
       <collision>
-        <geometry><mesh filename="package://leo_description/models/mycobot_280_pi/joint2.dae"/></geometry>
+        <geometry><mesh filename="package://leo_description/models/mycobot_280_pi/joint2.dae" scale="0.9 0.9 0.9"/></geometry>
         <origin xyz="0.0 0 -0.06096" rpy="0 0 -1.5708"/>
       </collision>
@@ -60,5 +60,5 @@
       <axis xyz="0 0 1"/>
       <limit effort="1000.0" lower="-2.9321" upper="2.9321" velocity="1.0"/>
-      <origin xyz="0 0 0.13956" rpy="0 0 0"/>
+      <origin xyz="0 0 0.13156" rpy="0 0 0"/>
       <parent link="${prefix}joint1"/>
       <child link="${prefix}joint2"/>
@@ -71,5 +71,5 @@
       </visual>
       <collision>
-        <geometry><mesh filename="package://leo_description/models/mycobot_280_pi/joint3.dae"/></geometry>
+        <geometry><mesh filename="package://leo_description/models/mycobot_280_pi/joint3.dae" scale="0.9 0.9 0.9"/></geometry>
         <origin xyz="0.0 0 0.03256" rpy="0 -1.5708 0"/>
       </collision>
@@ -79,5 +79,5 @@
       <axis xyz="0 0 1"/>
       <limit effort="1000.0" lower="-2.4434" upper="2.4434" velocity="1.0"/>
-      <origin xyz="0 0 -0.001" rpy="0 1.5708 -1.5708"/>
+      <origin xyz="0 0 -0.0" rpy="0 1.5708 -1.5708"/>
       <parent link="${prefix}joint2"/>
       <child link="${prefix}joint3"/>
@@ -90,5 +90,5 @@
       </visual>
       <collision>
-        <geometry><mesh filename="package://leo_description/models/mycobot_280_pi/joint4.dae"/></geometry>
+        <geometry><mesh filename="package://leo_description/models/mycobot_280_pi/joint4.dae" scale="0.9 0.9 0.9"/></geometry>
         <origin xyz="0.0 0 0.03056" rpy="0 -1.5708 0"/>
       </collision>
@@ -105,10 +105,10 @@
     <link name="${prefix}joint5">
       <visual>
-        <geometry><mesh filename="package://leo_description/models/mycobot_280_pi/J5_simple.stl"/></geometry>
-        <origin xyz="-0.02 0.002 0" rpy="0 0 0"/>
-      </visual>
-      <collision>
-        <geometry><mesh filename="package://leo_description/models/mycobot_280_pi/J5_simple.stl"/></geometry>
-        <origin xyz="-0.02 0.002 0" rpy="0 0 0"/>
+        <geometry><mesh filename="package://leo_description/models/mycobot_280_pi/joint5.dae"/></geometry>
+        <origin xyz="0.0 0 -0.03356" rpy="-1.5708 0 0"/>
+      </visual>
+      <collision>
+        <geometry><mesh filename="package://leo_description/models/mycobot_280_pi/joint5.dae" scale="0.9 0.9 0.9"/></geometry>
+        <origin xyz="0.0 0 -0.03356" rpy="-1.5708 0 0"/>
       </collision>
       <xacro:cylinder_inertial mass="0.1" radius="0.02" length="0.05"/>
@@ -128,5 +128,5 @@
       </visual>
       <collision>
-        <geometry><mesh filename="package://leo_description/models/mycobot_280_pi/joint6.dae"/></geometry>
+        <geometry><mesh filename="package://leo_description/models/mycobot_280_pi/joint6.dae" scale="0.9 0.9 0.9"/></geometry>
         <origin xyz="0 0.00 -0.038" rpy="0 0 0"/>
       </collision>
@@ -138,5 +138,5 @@
       <parent link="${prefix}joint5"/>
       <child link="${prefix}joint6"/>
-      <origin xyz="0 -0.07318 -0.001" rpy="1.5708 -1.5708 0"/>
+      <origin xyz="0 -0.07318 -0.0" rpy="1.5708 -1.5708 0"/>
       <dynamics damping="50.0" friction="50.0"/>
     </joint>
@@ -147,5 +147,5 @@
       </visual>
       <collision>
-        <geometry><mesh filename="package://leo_description/models/mycobot_280_pi/joint7.dae"/></geometry>
+        <geometry><mesh filename="package://leo_description/models/mycobot_280_pi/joint7.dae" scale="0.9 0.9 0.9"/></geometry>
         <origin xyz="0.0 0 -0.012" rpy="0 0 0"/>
       </collision>

Commit message: 更新机械臂

File: src/leo_description/urdf/mycobot_280_pi_adaptive_gripper.xacro (robot description, xacro)
@@ -374,4 +374,9 @@
         <state_interface name="velocity"/>
       </joint>
+      <joint name="${prefix}gripper_controller">
+        <command_interface name="position"/>
+        <state_interface name="position"/>
+        <state_interface name="velocity"/>
+      </joint>
     </ros2_control>
     <gazebo>

Commit message: 哈哈哈哈哈反正就是一大堆更新哈哈哈哈哈

File: src/leo_description/urdf/mycobot_280_pi_adaptive_gripper.xacro (robot description, xacro)
@@ -385,4 +385,39 @@
       </plugin>
     </gazebo>
+    <gazebo>
+      <plugin filename="gz-sim-mimic-joint-system" name="gz::sim::systems::MimicJoint">
+        <joint>${prefix}gripper_controller</joint>
+        <mimicJoint>${prefix}gripper_base_to_gripper_left2</mimicJoint>
+        <multiplier>1.0</multiplier>
+      </plugin>
+    </gazebo>
+    <gazebo>
+      <plugin filename="gz-sim-mimic-joint-system" name="gz::sim::systems::MimicJoint">
+        <joint>${prefix}gripper_controller</joint>
+        <mimicJoint>${prefix}gripper_left3_to_gripper_left1</mimicJoint>
+        <multiplier>-1.0</multiplier>
+      </plugin>
+    </gazebo>
+    <gazebo>
+      <plugin filename="gz-sim-mimic-joint-system" name="gz::sim::systems::MimicJoint">
+        <joint>${prefix}gripper_controller</joint>
+        <mimicJoint>${prefix}gripper_base_to_gripper_right3</mimicJoint>
+        <multiplier>-1.0</multiplier>
+      </plugin>
+    </gazebo>
+    <gazebo>
+      <plugin filename="gz-sim-mimic-joint-system" name="gz::sim::systems::MimicJoint">
+        <joint>${prefix}gripper_controller</joint>
+        <mimicJoint>${prefix}gripper_base_to_gripper_right2</mimicJoint>
+        <multiplier>-1.0</multiplier>
+      </plugin>
+    </gazebo>
+    <gazebo>
+      <plugin filename="gz-sim-mimic-joint-system" name="gz::sim::systems::MimicJoint">
+        <joint>${prefix}gripper_controller</joint>
+        <mimicJoint>${prefix}gripper_right3_to_gripper_right1</mimicJoint>
+        <multiplier>1.0</multiplier>
+      </plugin>
+    </gazebo>
   </xacro:macro>
 </robot>
